File: electronics/StepperDrive.kicad_pcb (KiCad board)
At the start: 2 copper layers, 58 x 33 mm, 40 parts, among them J1 USB_C_Receptacle_USB2.0_16P, J2 Screw_Terminal_01x04, J3 Barrel_Jack, J4 54602-908LF, J5 54602-908LF, J6 Conn_01x02, SW1 JS202011JCQN, U1 ATtiny814-SS, U2 TMC2209-LA, U3 FT231XS

Commit message: added GND Via for stall LED
Routing:
- net GND: vias 54 -> 55
Changed lines of the file:
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@@
+	)
+	(via
+		(at 69.4 53)
+		(size 0.6)
+		(drill 0.3)
+		(layers "F.Cu" "B.Cu")
+		(free yes)
+		(net 1)
 	)
 	(via
